Commit message: downgrade mini model, add varible foot position

File: mini_ros_simulation/robotis_mini_description/urdf/arm.urdf.xacro (robot description, xacro)
@@ -2,4 +2,21 @@
 <robot xmlns:xacro="http://ros.org/wiki/xacro">
   <xacro:macro name="robotis_mini_arm" params="side parent reflect">
+    <xacro:robotis_mini_servo_fixed name="${side}_shoulder" parent="${parent}"
+        xyz="0 -0.024 0" rpy="${(1-reflect)*M_PI/2} 0 ${(1+reflect)*M_PI/2}" initial_rotation="0" reflect="${reflect}"/>
+    <xacro:robotis_mini_dmfb03 name="${side}_biceps_anchor" parent="${side}_shoulder_link"
+        xyz="${reflect*0.012} 0 0.033" rpy="${M_PI/2} 0 ${reflect*-M_PI/2}" />
+    <xacro:robotis_mini_servo_rotating_with_wheel name="${side}_biceps" parent="${side}_biceps_anchor_link"
+        xyz="0 0 0" rpy="${M_PI/2} 0 ${reflect*M_PI/2}" initial_rotation="${reflect*M_PI/2.0}" reflect="${reflect}"/>
+    <xacro:robotis_mini_dmfb04 name="${side}_upper_arm" parent="${side}_biceps_link"
+        xyz="0 -0.045 0" rpy="${M_PI} ${reflect*-M_PI/2} 0" />
+    <xacro:robotis_mini_servo_rotating_with_wheel name="${side}_elbow" parent="${side}_upper_arm_link"
+        xyz="0 0 0" rpy="${M_PI} ${reflect*-M_PI/2} 0" initial_rotation="0" reflect="${reflect}"/>
+    <xacro:robotis_mini_spu5 name="${side}_lower_arm" parent="${side}_elbow_link"
+        xyz="0 -0.024 0" rpy="0 ${M_PI} ${M_PI}" />
+    <xacro:robotis_mini_spd3b3 name="${side}_wrist_anchor" parent="${side}_lower_arm_link"
+        xyz="0 0.0045 0" rpy="0 0 0" />
+    <xacro:robotis_mini_hand side="${side}" reflect="${reflect}" parent="${side}_wrist_anchor_link" />
+  </xacro:macro>
+  <xacro:macro name="robotis_mini_arm_upgrade" params="side parent reflect">
     <xacro:robotis_mini_servo_fixed name="${side}_shoulder" parent="${parent}"
         xyz="0 0 0" rpy="${(1-reflect)*M_PI/2} 0 ${(1+reflect)*M_PI/2}" initial_rotation="0" reflect="${reflect}"/>

File: mini_ros_simulation/robotis_mini_description/urdf/leg.urdf.xacro (robot description, xacro)
@@ -5,4 +5,34 @@
        xmlns:xacro="http://ros.org/wiki/xacro">
   <xacro:macro name="robotis_mini_leg" params="side parent reflect">
+    <xacro:robotis_mini_servo_fixed name="${side}_hip" parent="${parent}"
+        xyz="0 -0.024 0" rpy="0 0 ${M_PI}" initial_rotation="0" reflect="${-reflect}"/>
+    <xacro:robotis_mini_spd7v4 name="${side}_groin" parent="${side}_hip_link"
+        xyz="0 0 0.0165" rpy="${-M_PI/2} 0 ${-M_PI/2}" />
+    <xacro:robotis_mini_spd3b5 name="${side}_thigh_anchor" parent="${side}_groin_link"
+        xyz="0 -0.003 0" rpy="0 0 0" />
+    <xacro:robotis_mini_servo_fixed_with_wheel name="${side}_thigh" parent="${side}_thigh_anchor_link"
+        xyz="-0.006 -0.0135 0" rpy="${(1-reflect)*M_PI/2} 0 ${reflect*M_PI/2}" initial_rotation="0" reflect="${reflect}"/>
+    <xacro:robotis_mini_spu5 name="${side}_thigh_top" parent="${side}_thigh_servo_link"
+        xyz="0 -0.024 0" rpy="0 0 ${M_PI}" />
+    <xacro:robotis_mini_dmfb04 name="${side}_upper_leg" parent="${side}_thigh_link"
+        xyz="0 0 0" rpy="0 ${reflect*M_PI/2} ${M_PI}" />
+    <xacro:robotis_mini_servo_fixed_with_wheel name="${side}_knee" parent="${side}_upper_leg_link"
+        xyz="0 -0.045 0" rpy="${M_PI} ${reflect*M_PI/2} 0" initial_rotation="0" reflect="${reflect}"/>
+    <xacro:robotis_mini_dmfb05 name="${side}_lower_leg" parent="${side}_knee_link"
+        xyz="0 0 0" rpy="${-M_PI/2} ${reflect*M_PI/2} 0" />
+    <xacro:robotis_mini_servo_rotating_with_wheel name="${side}_ankle" parent="${side}_lower_leg_link"
+        xyz="0 0 0.042" rpy="${M_PI/2} 0 ${reflect*-M_PI/2}" initial_rotation="0" reflect="${reflect}"/>
+    <xacro:robotis_mini_spd3b7 name="${side}_achiles" parent="${side}_ankle_link"
+        xyz="${reflect*0.0135} -0.009 0" rpy="${(1+reflect)*M_PI/2} 0 ${M_PI/2}" />
+    <xacro:robotis_mini_spd7v4 name="${side}_foot_anchor" parent="${side}_achiles_link"
+        xyz="0.006 0.003 0" rpy="0 0 0" />
+    <xacro:robotis_mini_servo_rotating name="${side}_foot" parent="${side}_foot_anchor_link"
+        xyz="0 0.0165 0" rpy="${M_PI/2} ${(1+reflect)*M_PI/2} 0" initial_rotation="0" reflect="${reflect}"/>
+    <xacro:robotis_mini_dmfb06 name="${side}_forefoot" parent="${side}_foot_link"
+        xyz="${reflect*-0.03} -0.009 0" rpy="0 0 ${reflect*-M_PI/2}" />
+    <xacro:robotis_mini_dmfb07 name="${side}_sole" parent="${side}_forefoot_link"
+        xyz="0 0 0.03" rpy="0 0 0" />
+  </xacro:macro>
+  <xacro:macro name="robotis_mini_leg_upgrade" params="side parent reflect">
     <xacro:robotis_mini_servo_fixed name="${side}_hip" parent="${parent}"
         xyz="0 0 0" rpy="0 0 ${M_PI}" initial_rotation="0" reflect="${-reflect}"/>

File: mini_ros_simulation/robotis_mini_description/urdf/robotis_mini.urdf.xacro (robot description, xacro)
@@ -14,9 +14,14 @@
   <xacro:include filename="$(find robotis_mini_description)/urdf/leg.urdf.xacro" />
   <xacro:robotis_mini_base name="base"/>
-  <xacro:robotis_mini_body2 parent="base_link" />
+  <!-- <xacro:robotis_mini_body2 parent="base_link" />
   <xacro:robotis_mini_arm side="l" reflect="1" parent="left_arm_socket_link" />
   <xacro:robotis_mini_arm side="r" reflect="-1" parent="right_arm_socket_link" />
   <xacro:robotis_mini_leg side="l" reflect="1" parent="left_leg_socket_link" />
-  <xacro:robotis_mini_leg side="r" reflect="-1" parent="right_leg_socket_link" />
+  <xacro:robotis_mini_leg side="r" reflect="-1" parent="right_leg_socket_link" /> -->
+  <xacro:robotis_mini_body parent="base_link" />
+  <xacro:robotis_mini_arm side="l" reflect="1" parent="l_shoulder_anchor_link" />
+  <xacro:robotis_mini_arm side="r" reflect="-1" parent="r_shoulder_anchor_link" />
+  <xacro:robotis_mini_leg side="l" reflect="1" parent="l_hip_anchor_link" />
+  <xacro:robotis_mini_leg side="r" reflect="-1" parent="r_hip_anchor_link" />
   <gazebo>
     <plugin name="gazebo_ros_control" filename="libgazebo_ros_control.so">
